File: Relais-Karte.kicad_pcb (KiCad board)
At the start: 2 copper layers, 38.5 x 74.5 mm, 8 parts, among them J1 MKDS_3-2_5.08, J2 MKDS_3-2_5.08, J3 MKDS_3-3_5.08, J4 MKDS_3-2_5.08, K1 G2RL-1-E, SW1 L101011MS02Q

Commit message: wip
Other:
- board text added: "GND"
Changed lines of the file:
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@@
 	(gr_rect
 		(start 113.25 86)
-		(end 127 95.5)
+		(end 131 95.5)
 		(stroke
 			(width 0.1)
@@
 		(layer "Edge.Cuts")
 	)
+	(gr_text "GND"
+		(at 125.5 112 0)
+		(layer "F.SilkS")
+		(effects
+			(font
+				(size 1 1)
+				(thickness 0.1)
+			)
+			(justify left bottom)
+		)
+	)
 	(gr_text "NC NO GND"
