File: Relais-Karte.kicad_pcb (KiCad board)
At the start: 2 copper layers, 38.5 x 77 mm, 24 parts, among them J1 MKDS_3-2_5.08, J2 MKDS_3-2_5.08, J3 MKDS_3-3_5.08, J4 MKDS_3-2_5.08, K1 G2RL-1-E, Q1 BC846, Q2 BC846, SW1 L101011MS02Q, U1 TL431DBZ, U2 TL431DBZ

Commit message: final version
Other:
- board text removed: "${COMMENT1}"
- board text removed: "${COMMENT2}"
- board text removed: "${COMMENT3}"
- board text removed: "${COMMENT4}"
- board text removed: "${COMPANY}"
- board text removed: "${ISSUE_DATE}"
- board text removed: "${REVISION}"
- board text removed: "${TITLE}"
