File: Relais-Karte.kicad_sch (KiCad schematic)
At the start: 10 parts, among them J1 MKDS_3-2_5.08, J2 MKDS_3-2_5.08, J3 MKDS_3-3_5.08, J4 MKDS_3-2_5.08, K1 G2RL-1-E, M1 Motor_DC, SW1 L101011MS02Q, SW2 SW_SPST

Commit message: wip
Parts:
- F1: LCSC (none) -> C19727304
- J1, J2, J4: LCSC (none) -> C475092
- J3: LCSC (none) -> C475093
Changed lines of the file:
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@@
 			)
 		)
-		(property "LCSC" ""
+		(property "LCSC" "C475092"
 			(at 115.57 92.71 0)
 			(effects
@@
 		)
 		(property "Digikey" "277-1027-ND"
+			(at 58.42 52.07 0)
+			(effects
+				(font
+					(size 1.27 1.27)
+				)
+				(hide yes)
+			)
+		)
+		(property "LCSC" "C475092"
+			(at 58.42 52.07 0)
+			(effects
+				(font
+					(size 1.27 1.27)
+				)
+				(hide yes)
+			)
+		)
+		(property "Mouser" ""
 			(at 58.42 52.07 0)
 			(effects
@@
 			)
 		)
-		(property "LCSC" ""
+		(property "LCSC" "C19727304"
 			(at 81.28 39.37 0)
 			(effects
@@
 		)
 		(instances
-			(project ""
+			(project "Relais-Karte"
 				(path "/c7fa4b37-882c-44ba-bde7-299b1a97af71"
 					(reference "F1")
@@
 			)
 		)
+		(property "LCSC" "C475092"
+			(at 58.42 41.91 0)
+			(effects
+				(font
+					(size 1.27 1.27)
+				)
+				(hide yes)
+			)
+		)
+		(property "Mouser" ""
+			(at 58.42 41.91 0)
+			(effects
+				(font
+					(size 1.27 1.27)
+				)
+				(hide yes)
+			)
+		)
 		(pin "2"
 		)
@@
 		)
 		(instances
-			(project ""
+			(project "Relais-Karte"
 				(path "/c7fa4b37-882c-44ba-bde7-299b1a97af71"
 					(reference "J1")
@@
 		)
 		(instances
-			(project ""
+			(project "Relais-Karte"
 				(path "/c7fa4b37-882c-44ba-bde7-299b1a97af71"
 					(reference "D1")
@@
 		)
 		(instances
-			(project ""
+			(project "Relais-Karte"
 				(path "/c7fa4b37-882c-44ba-bde7-299b1a97af71"
 					(reference "K1")
@@
 			)
 		)
+		(property "LCSC" "C475093"
+			(at 58.42 72.39 0)
+			(effects
+				(font
+					(size 1.27 1.27)
+				)
+				(hide yes)
+			)
+		)
+		(property "Mouser" ""
+			(at 58.42 72.39 0)
+			(effects
+				(font
+					(size 1.27 1.27)
+				)
+				(hide yes)
+			)
+		)
 		(pin "3"
 		)
@@
 		)
 		(instances
-			(project ""
+			(project "Relais-Karte"
 				(path "/c7fa4b37-882c-44ba-bde7-299b1a97af71"
 					(reference "J3")
@@
 		)
 		(instances
-			(project ""
+			(project "Relais-Karte"
 				(path "/c7fa4b37-882c-44ba-bde7-299b1a97af71"
 					(reference "SW1")
