File: Relais-Karte.kicad_sch (KiCad schematic)
At the start: 22 parts, among them J1 MKDS_3-2_5.08, J2 MKDS_3-2_5.08, J3 MKDS_3-3_5.08, J4 MKDS_3-2_5.08, K1 G2RL-1-E, M1 Motor_DC, Q1 BC846, Q2 BC846, SW1 L101011MS02Q, SW2 SW_SPST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

Commit message: led typ angepasst
Parts:
- D2, D3: value KPTD-3216SECK -> KPTD-3216ZGCK
Changed lines of the file:
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@@
 			)
 		)
-		(property "Value" "KPTD-3216SECK"
+		(property "Value" "KPTD-3216ZGCK"
 			(at 215.9 86.6774 90)
 			(effects
@@
 			)
 		)
-		(property "Value" "KPTD-3216SECK"
+		(property "Value" "KPTD-3216ZGCK"
 			(at 215.9 60.0074 90)
 			(effects
