File: Relais-Karte.kicad_sch (KiCad schematic)
At the start: 24 parts, among them J1 MKDS_3-2_5.08, J2 MKDS_3-2_5.08, J3 MKDS_3-3_5.08, J4 MKDS_3-2_5.08, K1 G2RL-1-E, Q1 BC846, Q2 BC846, SW1 L101011MS02Q, U1 TL431DBZ, U2 TL431DBZ

Commit message: final version
Parts:
- PCB1, Repo1: value ~ -> (none)
