File: Relais-Karte/source_2026-03-21/Relais-Karte.kicad_sch (KiCad schematic)
At the start: 20 parts, among them J1 MKDS_3-2_5.08, J2 MKDS_3-2_5.08, J3 MKDS_3-3_5.08, J4 MKDS_3-2_5.08, K1 G2RL-1-E, M1 Motor_DC, Q1 BC846, Q2 BC846, SW1 L101011MS02Q, SW2 SW_SPST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

Commit message: leds added
Parts:
- D2, D3: symbol Symbols:LED -> _PS_LIB:LED
- Q1, Q2: symbol Symbols:BC846 -> Transistor_BJT:BC846
- R1, R4: symbol Symbols:Resistor 22K -> Resistor_E12_0603:Resistor 22K
- R2, R3: symbol Symbols:Resistor 270R -> Resistor_E12_0603:Resistor 270R
- U1, U2: symbol Symbols:TL431DBZ -> Reference_Voltage:TL431DBZ
Changed lines of the file:
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@@
 	)
 	(symbol
-		(lib_id "Symbols:TL431DBZ")
+		(lib_id "Reference_Voltage:TL431DBZ")
 		(at 193.04 62.23 0)
 		(mirror y)
@@
 	)
 	(symbol
-		(lib_id "Symbols:Resistor 22K")
+		(lib_id "Resistor_E12_0603:Resistor 22K")
 		(at 168.91 57.15 0)
 		(unit 1)
@@
 	)
 	(symbol
-		(lib_id "Symbols:Resistor 270R")
+		(lib_id "Resistor_E12_0603:Resistor 270R")
 		(at 199.39 52.07 90)
 		(unit 1)
@@
 	)
 	(symbol
-		(lib_id "Symbols:Resistor 270R")
+		(lib_id "Resistor_E12_0603:Resistor 270R")
 		(at 199.39 78.74 90)
 		(unit 1)
@@
 	)
 	(symbol
-		(lib_id "Symbols:BC846")
+		(lib_id "Transistor_BJT:BC846")
 		(at 182.88 54.61 90)
 		(unit 1)
@@
 	)
 	(symbol
-		(lib_id "Symbols:LED")
+		(lib_id "_PS_LIB:LED")
 		(at 212.09 83.82 90)
 		(unit 1)
@@
 	)
 	(symbol
-		(lib_id "Symbols:LED")
+		(lib_id "_PS_LIB:LED")
 		(at 212.09 57.15 90)
 		(unit 1)
@@
 	)
 	(symbol
-		(lib_id "Symbols:TL431DBZ")
+		(lib_id "Reference_Voltage:TL431DBZ")
 		(at 193.04 88.9 0)
 		(mirror y)
@@
 	)
 	(symbol
-		(lib_id "Symbols:Resistor 22K")
+		(lib_id "Resistor_E12_0603:Resistor 22K")
 		(at 168.91 83.82 0)
 		(unit 1)
@@
 	)
 	(symbol
-		(lib_id "Symbols:BC846")
+		(lib_id "Transistor_BJT:BC846")
 		(at 182.88 81.28 90)
 		(unit 1)

Commit message: wip
Parts:
- added PCB1: ~, _PS_LIB_PCB:_PCB, symbol _PS_LIB:_PCB
- added Repo1: ~, _PS_LIB_PCB:_Repository, symbol _PS_LIB:_Repository
- D2, D3: symbol _PS_LIB:LED -> Symbols:LED
- Q1, Q2: symbol Transistor_BJT:BC846 -> Symbols:BC846
- R1, R4: symbol Resistor_E12_0603:Resistor 22K -> Symbols:Resistor 22K
- R2, R3: symbol Resistor_E12_0603:Resistor 270R -> Symbols:Resistor 270R
- U1, U2: symbol Reference_Voltage:TL431DBZ -> Symbols:TL431DBZ
Changed lines of the file:
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@@
 	)
 	(symbol
-		(lib_id "Reference_Voltage:TL431DBZ")
+		(lib_id "_PS_LIB:_PCB")
+		(at 177.8 165.1 0)
+		(unit 1)
+		(exclude_from_sim yes)
+		(in_bom no)
+		(on_board yes)
+		(dnp no)
+		(property "Reference" "PCB1"
+			(at 177.8 161.29 0)
+			(effects
+				(font
+					(size 1.27 1.27)
+				)
+				(justify left bottom)
+			)
+		)
+		(property "Value" "~"
+			(at 177.8 165.1 0)
+			(effects
+				(font
+					(size 1.27 1.27)
+				)
+				(hide yes)
+			)
+		)
+		(property "Footprint" "_PS_LIB_PCB:_PCB"
+			(at 186.944 163.83 0)
+			(effects
+				(font
+					(size 1.27 1.27)
+				)
+				(hide yes)
+			)
+		)
+		(property "Datasheet" ""
+			(at 177.8 165.1 0)
+			(effects
+				(font
+					(size 1.27 1.27)
+				)
+				(hide yes)
+			)
+		)
+		(property "Description" ""
+			(at 177.8 165.1 0)
+			(effects
+				(font
+					(size 1.27 1.27)
+				)
+				(hide yes)
+			)
+		)
+		(property "LCSC" ""
+			(at 177.8 165.1 0)
+			(effects
+				(font
+					(size 1.27 1.27)
+				)
+				(hide yes)
+			)
+		)
+		(property "Digikey" ""
+			(at 177.8 165.1 0)
+			(effects
+				(font
+					(size 1.27 1.27)
+				)
+				(hide yes)
+			)
+		)
+		(property "Mouser" ""
+			(at 177.8 165.1 0)
+			(effects
+				(font
+					(size 1.27 1.27)
+				)
+				(hide yes)
+			)
+		)
+		(instances
+			(project "Relais-Karte"
+				(path "/c7fa4b37-882c-44ba-bde7-299b1a97af71"
+					(reference "PCB1")
+					(unit 1)
+				)
+			)
+		)
+	)
+	(symbol
+		(lib_id "Symbols:TL431DBZ")
 		(at 193.04 62.23 0)
 		(mirror y)
@@
 	)
 	(symbol
-		(lib_id "Resistor_E12_0603:Resistor 22K")
+		(lib_id "Symbols:Resistor 22K")
 		(at 168.91 57.15 0)
 		(unit 1)
@@
 	)
 	(symbol
-		(lib_id "Resistor_E12_0603:Resistor 270R")
+		(lib_id "Symbols:Resistor 270R")
 		(at 199.39 52.07 90)
 		(unit 1)
@@
 	)
 	(symbol
-		(lib_id "Resistor_E12_0603:Resistor 270R")
+		(lib_id "_PS_LIB:_Repository")
+		(at 207.01 165.1 0)
+		(unit 1)
+		(exclude_from_sim yes)
+		(in_bom no)
+		(on_board yes)
+		(dnp no)
+		(fields_autoplaced yes)
+		(property "Reference" "Repo1"
+			(at 213.487 160.02 0)
+			(effects
+				(font
+					(size 1.27 1.27)
+				)
+			)
+		)
+		(property "Value" "~"
+			(at 207.01 165.1 0)
+			(effects
+				(font
+					(size 1.27 1.27)
+				)
+				(hide yes)
+			)
+		)
+		(property "Footprint" "_PS_LIB_PCB:_Repository"
+			(at 216.154 163.83 0)
+			(effects
+				(font
+					(size 1.27 1.27)
+				)
+				(hide yes)
+			)
+		)
+		(property "Datasheet" ""
+			(at 207.01 165.1 0)
+			(effects
+				(font
+					(size 1.27 1.27)
+				)
+				(hide yes)
+			)
+		)
+		(property "Description" ""
+			(at 207.01 165.1 0)
+			(effects
+				(font
+					(size 1.27 1.27)
+				)
+				(hide yes)
+			)
+		)
+		(instances
+			(project "Relais-Karte"
+				(path "/c7fa4b37-882c-44ba-bde7-299b1a97af71"
+					(reference "Repo1")
+					(unit 1)
+				)
+			)
+		)
+	)
+	(symbol
+		(lib_id "Symbols:Resistor 270R")
 		(at 199.39 78.74 90)
 		(unit 1)
@@
 	)
 	(symbol
-		(lib_id "Transistor_BJT:BC846")
+		(lib_id "Symbols:BC846")
 		(at 182.88 54.61 90)
 		(unit 1)
@@
 	)
 	(symbol
-		(lib_id "_PS_LIB:LED")
+		(lib_id "Symbols:LED")
 		(at 212.09 83.82 90)
 		(unit 1)
@@
 	)
 	(symbol
-		(lib_id "_PS_LIB:LED")
+		(lib_id "Symbols:LED")
 		(at 212.09 57.15 90)
 		(unit 1)
@@
 	)
 	(symbol
-		(lib_id "Reference_Voltage:TL431DBZ")
+		(lib_id "Symbols:TL431DBZ")
 		(at 193.04 88.9 0)
 		(mirror y)
@@
 	)
 	(symbol
-		(lib_id "Resistor_E12_0603:Resistor 22K")
+		(lib_id "Symbols:Resistor 22K")
 		(at 168.91 83.82 0)
 		(unit 1)
@@
 	)
 	(symbol
-		(lib_id "Transistor_BJT:BC846")
+		(lib_id "Symbols:BC846")
 		(at 182.88 81.28 90)
 		(unit 1)
